File: hw/hw.kicad_pcb (KiCad board)
At the start: 2 copper layers, 38 parts, among them J1 Pi Operating Voltage, J2 Pi LED Signals In, J3 Pi Button Signals Out, J4 Laser Turret Signals In, J5 Mouse Servo Signal In, J6 Fan Signal In, M1 Yaw, M2 Pitch, M3 Mouse, M4 Fan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

Commit message: Created pcb layout
Parts:
- moved J4 107.8 mm to (91.4, 109.2), turned to 90 degrees
- moved R10 103.6 mm to (104.1, 100.3), turned to 270 degrees
- moved J3 96.0 mm to (96.5, 83.8), turned to 90 degrees
- moved J2 92.3 mm to (96.5, 88.9), turned to 90 degrees
- moved J5 88.2 mm to (85.1, 109.2), turned to 270 degrees
- moved R9 87.6 mm to (77.5, 105.4)
- moved M1 87.2 mm to (94.0, 101.6), turned to 90 degrees
- moved R11 85.8 mm to (102.9, 68.6), turned to 180 degrees
- moved M2 84.7 mm to (94.0, 104.1), turned to 90 degrees
- moved Q5 83.8 mm to (106.7, 68.6), turned to 270 degrees
- moved D5 82.8 mm to (95.2, 72.4)
- moved D4 80.7 mm to (99.1, 99.1), turned to 270 degrees
- moved M3 79.5 mm to (94.0, 96.5), turned to 90 degrees
- moved R8 79.4 mm to (77.5, 99.1)
- moved R4 78.7 mm to (86.4, 86.4), turned to 180 degrees
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Routing:
- net +5V: track 0.00 -> 108.1 mm
- net Net-(J6-Pad1): track 0.00 -> 32.4 mm
- net Net-(C3-Pad1): track 0.00 -> 29.8 mm
- net Net-(C2-Pad1): track 0.00 -> 26.2 mm
- net Net-(J2-Pad3): track 0.00 -> 25.6 mm
- net Net-(D5-Pad2): track 0.00 -> 23.6 mm
- net Net-(C1-Pad1): track 0.00 -> 22.6 mm
- net Net-(J2-Pad2): track 0.00 -> 18.9 mm
- net +3V3: track 0.00 -> 17.8 mm
- net Net-(J5-Pad1): track 0.00 -> 16.4 mm
- net Net-(J2-Pad1): track 0.00 -> 13.0 mm
- net Net-(D4-Pad1): track 0.00 -> 10.8 mm
- net Net-(J4-Pad1): track 0.00 -> 9.46 mm
- net Net-(J4-Pad3): track 0.00 -> 9.39 mm
- net Net-(D3-Pad1): track 0.00 -> 9.03 mm
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- added copper zone on B.Cu, net GND
Other:
- board outline added: 57.1 x 52.1 mm
- net class Default: clearance 0.2 -> 0.4; trace_width 0.25 -> 0.5; via_dia 0.8 -> 1.6
- rule trace_clearance: 0.2 -> 0.4
